File: pcb/nz/nz.kicad_sch (KiCad schematic)
At the start: 90 parts, among them J1 USB_C_Receptacle_USB2.0_16P, J10 RC522_1, J11 MCP2515_EXP, J12 Conn_02x02, J13 Conn_01x04, J14 2601-1106, J2 Conn_01x04, J3 2601-1103, J5 Conn_01x04, J6 Conn_02x12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

Commit message: ipdate
Parts:
- added CAN_TERM1: SW_DIP_x01, Button_Switch_SMD:SW_DIP_SPSTx01_Slide_6.7x4.1mm_W6.73mm_P2.54mm_LowProfile_JPin, symbol Switch:SW_DIP_x01
- added R22: R120, Resistor_SMD:R_0402_1005Metric, symbol Device:R
- renumbered SW2 to EN1, SW3 to IO0
Connections:
- net +3.3V: no longer C11.1, C12.1, J2.2 (Pin_2), J5.2 (Pin_2), R11.2, R12.2
- net +3.3V Sensor: now also C11.1, C12.1, J2.2 (Pin_2), J5.2 (Pin_2), R11.2, R12.2
- net +5V: no longer U3.5 (VBUS)
- net +5VA: now also U3.5 (VBUS)
- net CAN_H: now also CAN_TERM1.2
- net CAN_L: now also R22.2
- new net: CAN_TERM1.1, R22.1
Other:
- moved on the sheet: C14, C15, C16, F2, J14, R16, U1
