File: pcb/nz/nz.kicad_pcb (KiCad board)
At the start: 6 copper layers, 90 parts, among them J1 USB_C_Receptacle_USB2.0_16P, J10 RC522_1, J11 MCP2515_EXP, J12 Conn_02x02, J13 Conn_01x04, J14 2601-1106, J2 Conn_01x04, J3 2601-1103, J5 Conn_01x04, J6 Conn_02x12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

Commit message: ipdate
Parts:
- added CAN_TERM1: SW_DIP_x01, Button_Switch_SMD:SW_DIP_SPSTx01_Slide_6.7x4.1mm_W6.73mm_P2.54mm_LowProfile_JPin, F.Cu at (106.5, 121.1)
- added R22: R120, Resistor_SMD:R_0402_1005Metric, F.Cu at (112.9, 114.3)
- moved Q2 22.3 mm to (167.9, 89.2)
- moved R13 22.3 mm to (165.4, 89.1)
- moved R14 22.3 mm to (164.4, 89.1)
- moved C6 14.3 mm to (120.8, 100.2)
- moved D6 5.52 mm to (111.7, 104.2)
- moved C27 4.06 mm to (125.4, 108.0)
- moved R19 3.62 mm to (127.2, 109.1), turned to 90 degrees
- moved R20 3.18 mm to (127.2, 111.1), turned to 90 degrees
- moved C24 3.15 mm to (112.8, 108.2), turned to -90 degrees
- moved C23 2.44 mm to (113.4, 108.2), turned to -90 degrees
- moved U3 2.05 mm to (108.0, 98.0), turned to 180 degrees
- moved F1 1.90 mm to (103.4, 98.3)
- moved C22 1.85 mm to (114.0, 108.2), turned to -90 degrees
- moved FB1 1.58 mm to (99.3, 97.6)
- moved C21 1.54 mm to (114.6, 108.2), turned to -90 degrees
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- renumbered SW2 to EN1, SW3 to IO0
Connections:
- C11 pad 1: +3.3V -> +3.3V Sensor
- C12 pad 1: +3.3V -> +3.3V Sensor
- J2 pad 2: +3.3V -> +3.3V Sensor
- J5 pad 2: +3.3V -> +3.3V Sensor
- R11 pad 2: +3.3V -> +3.3V Sensor
- R12 pad 2: +3.3V -> +3.3V Sensor
- U3 pad 5: +5V -> +5VA
Routing:
- net GND: track 5.00 -> 91.8 mm
- net /CAN_H: track 0.00 -> 59.0 mm
- net /CAN_L: track 0.00 -> 31.1 mm
- net Net-(J3-1_1): track 26.4 -> 0.00 mm
- net Net-(J3-3_1): track 26.4 -> 0.00 mm
- net +5V: track 0.00 -> 23.4 mm, vias 0 -> 2
- net +5VP: track 0.00 -> 19.5 mm, vias 0 -> 2
- net Net-(J3-2_1): track 11.2 -> 0.00 mm
- net Net-(CAN_TERM1-Pad1): track 0.00 -> 7.59 mm
- net Net-(J14-1_1): track 5.00 -> 10.6 mm
- net Net-(D6-K): track 0.00 -> 4.02 mm
- net Net-(J1-CC1): track 0.00 -> 2.71 mm
- net Net-(F1-Pad1): track 0.00 -> 2.67 mm
- net +5VA: track 0.00 -> 2.34 mm
- net +12V: track 0.00 -> 2.20 mm
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- removed copper zone on B.Cu, net GND
Other:
- board outline added: 100 x 50 mm
- board text added: "+"
- board text added: "-"
- board text added: "COM"
- board text added: "H"
- board text added: "L"
- board text added: "NC"
- board text added: "NO"

Commit message: started addressable led
Parts:
- moved Q1 99.8 mm to (219.8, 102.7)
- moved C3 99.2 mm to (210.7, 94.9), turned to 0 degrees
- moved C4 98.8 mm to (210.7, 96.5), turned to 0 degrees
- moved C2 98.6 mm to (210.7, 93.2), turned to 0 degrees
- moved C5 98.2 mm to (210.7, 98.2), turned to 0 degrees
- moved C1 97.9 mm to (210.7, 91.6), turned to 0 degrees
- moved J12 93.2 mm to (216.4, 96.3), turned to 0 degrees
- moved R4 92.9 mm to (213.2, 95.7)
- moved R5 92.8 mm to (213.2, 97.7)
- moved J7 92.2 mm to (216.4, 92.3), turned to 0 degrees
- moved C6 89.8 mm to (210.7, 99.8)
- moved L1 89.6 mm to (214.2, 105.9)
- moved J6 68.5 mm to (206.8, 92.3), turned to 0 degrees
- moved F1 15.7 mm to (116.6, 89.8)
- moved FB1 15.1 mm to (112.2, 89.8), turned to 0 degrees
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Routing:
- net /CAN_H: track 59.0 -> 0.00 mm
- net GND: track 91.8 -> 34.8 mm
- net /RELAY: track 0.00 -> 40.4 mm, vias 0 -> 2
- net +3.3V: track 0.00 -> 31.4 mm, vias 0 -> 3
- net /CAN_L: track 31.1 -> 0.00 mm
- net /LED_B: track 0.00 -> 26.4 mm, vias 0 -> 2
- net +5V: track 23.4 -> 0.00 mm, vias 2 -> 0
- net /LED_R: track 0.00 -> 20.3 mm, vias 0 -> 2
- net /LED_G: track 0.00 -> 15.2 mm, vias 0 -> 2
- net /MOSI: track 0.00 -> 12.6 mm
- net Net-(J14-1_1): track 10.6 -> 0.00 mm
- net Net-(J1-D--PadA7): track 0.00 -> 9.17 mm, vias 0 -> 2
- net Net-(CAN_TERM1-Pad1): track 7.59 -> 0.00 mm
- net /SCK: track 0.00 -> 5.21 mm
- net /MISO: track 0.00 -> 4.91 mm
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